File: sch_and_pcb/epm3032_ym2149x2.kicad_sch (KiCad schematic)
At the start: 17 parts, among them U1 YM2149, U2 YM2149, U3 AMS1117-3.3, U4 NE5532, X1 zx-bus

Commit message: >> продолжаем продолжать. Макетка рулез.
Connections:
- net +5V: now also U1.28 (BC2), U1.40 (VCC), U2.28 (BC2), U2.40 (VCC)
- net GND: now also U1.1 (VSS), U1.24 (~{A9}), U2.1 (VSS), U2.24 (~{A9})
- net a1: no longer D1.4 (io)
- net d1: now also D1.28 (io); no longer D1.36 (io)
- net wr: now also D1.12 (io); no longer D1.7 (tdi)
- net a0: now reaches D1.11 (io)
- net a0: now also X1.40 (A0)
- net beeper: now reaches D1.21 (io)
- net tapeout: now reaches D1.24 (io)
- no-connect marks 0 -> 4
Changed lines of the file:
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@@
   (junction (at 44.45 72.39) (diameter 0) (color 0 0 0 0)
   )
+  (no_connect (at 176.53 78.74))
+  (no_connect (at 176.53 68.58))
+  (no_connect (at 232.41 68.58))
+  (no_connect (at 232.41 78.74))
   (bus_entry (at 219.71 68.58) (size 2.54 -2.54)
     (stroke (width 0) (type default) (color 0 0 0 0))
@@
     (stroke (width 0) (type default) (color 0 0 0 0))
   )
-  (bus_entry (at 163.83 71.12) (size 2.54 -2.54)
-    (stroke (width 0) (type default) (color 0 0 0 0))
-  )
   (bus_entry (at 54.61 125.73) (size 2.54 -2.54)
     (stroke (width 0) (type default) (color 0 0 0 0))
@@
     (stroke (width 0) (type default) (color 0 0 0 0))
   )
+  (bus_entry (at 85.09 121.92) (size 2.54 -2.54)
+    (stroke (width 0) (type default) (color 0 0 0 0))
+  )
   (bus_entry (at 54.61 146.05) (size 2.54 -2.54)
     (stroke (width 0) (type default) (color 0 0 0 0))
@@
     (stroke (width 0) (type default) (color 0 0 0 0))
   )
+  (bus_entry (at 186.69 92.71) (size 2.54 -2.54)
+    (stroke (width 0) (type default) (color 0 0 0 0))
+  )
   (bus_entry (at 163.83 40.64) (size 2.54 -2.54)
     (stroke (width 0) (type default) (color 0 0 0 0))
@@
     (stroke (width 0) (type default) (color 0 0 0 0))
   )
-  (bus_entry (at 161.29 55.88) (size 2.54 2.54)
+  (bus_entry (at 242.57 92.71) (size 2.54 -2.54)
     (stroke (width 0) (type default) (color 0 0 0 0))
   )
@@
     (stroke (width 0) (type default) (color 0 0 0 0))
   )
-  (bus_entry (at 219.71 71.12) (size 2.54 -2.54)
-    (stroke (width 0) (type default) (color 0 0 0 0))
-  )
   (bus_entry (at 163.83 73.66) (size 2.54 -2.54)
     (stroke (width 0) (type default) (color 0 0 0 0))
@@
     (stroke (width 0) (type default) (color 0 0 0 0))
   )
-  (bus (pts (xy 219.71 71.12) (xy 219.71 73.66))
+  (bus (pts (xy 219.71 68.58) (xy 219.71 73.66))
     (stroke (width 0) (type default) (color 0 0 0 0))
   )
@@
     (stroke (width 0) (type default) (color 0 0 0 0))
   )
-  (wire (pts (xy 146.05 55.88) (xy 161.29 55.88))
-    (stroke (width 0) (type default) (color 0 0 0 0))
-  )
   (bus (pts (xy 87.63 172.72) (xy 87.63 179.07))
     (stroke (width 0) (type default) (color 0 0 0 0))
@@
     (stroke (width 0) (type default) (color 0 0 0 0))
   )
+  (bus (pts (xy 186.69 92.71) (xy 219.71 92.71))
+    (stroke (width 0) (type default) (color 0 0 0 0))
+  )
   (wire (pts (xy 90.17 66.04) (xy 105.41 66.04))
     (stroke (width 0) (type default) (color 0 0 0 0))
@@
     (stroke (width 0) (type default) (color 0 0 0 0))
   )
-  (bus (pts (xy 87.63 27.94) (xy 87.63 30.48))
-    (stroke (width 0) (type default) (color 0 0 0 0))
-  )
   (bus (pts (xy 25.4 57.15) (xy 25.4 62.23))
     (stroke (width 0) (type default) (color 0 0 0 0))
@@
     (stroke (width 0) (type default) (color 0 0 0 0))
   )
+  (bus (pts (xy 87.63 119.38) (xy 87.63 121.92))
+    (stroke (width 0) (type default) (color 0 0 0 0))
+  )
   (bus (pts (xy 87.63 55.88) (xy 87.63 58.42))
     (stroke (width 0) (type default) (color 0 0 0 0))
@@
     (stroke (width 0) (type default) (color 0 0 0 0))
   )
-  (wire (pts (xy 166.37 68.58) (xy 176.53 68.58))
-    (stroke (width 0) (type default) (color 0 0 0 0))
-  )
   (bus (pts (xy 219.71 73.66) (xy 219.71 92.71))
     (stroke (width 0) (type default) (color 0 0 0 0))
   )
-  (bus (pts (xy 87.63 30.48) (xy 87.63 33.02))
-    (stroke (width 0) (type default) (color 0 0 0 0))
-  )
   (wire (pts (xy 27.94 38.1) (xy 44.45 38.1))
     (stroke (width 0) (type default) (color 0 0 0 0))
@@
     (stroke (width 0) (type default) (color 0 0 0 0))
   )
-  (bus (pts (xy 163.83 92.71) (xy 219.71 92.71))
+  (bus (pts (xy 163.83 92.71) (xy 186.69 92.71))
     (stroke (width 0) (type default) (color 0 0 0 0))
   )
@@
     (stroke (width 0) (type default) (color 0 0 0 0))
   )
-  (bus (pts (xy 87.63 33.02) (xy 87.63 35.56))
+  (bus (pts (xy 87.63 27.94) (xy 87.63 35.56))
+    (stroke (width 0) (type default) (color 0 0 0 0))
+  )
+  (wire (pts (xy 189.23 86.36) (xy 189.23 90.17))
     (stroke (width 0) (type default) (color 0 0 0 0))
   )
@@
     (stroke (width 0) (type default) (color 0 0 0 0))
   )
-  (bus (pts (xy 87.63 116.84) (xy 87.63 121.92))
+  (bus (pts (xy 87.63 116.84) (xy 87.63 119.38))
     (stroke (width 0) (type default) (color 0 0 0 0))
   )
@@
     (stroke (width 0) (type default) (color 0 0 0 0))
   )
+  (bus (pts (xy 242.57 92.71) (xy 269.24 92.71))
+    (stroke (width 0) (type default) (color 0 0 0 0))
+  )
   (bus (pts (xy 163.83 68.58) (xy 163.83 71.12))
     (stroke (width 0) (type default) (color 0 0 0 0))
@@
     (stroke (width 0) (type default) (color 0 0 0 0))
   )
-  (wire (pts (xy 222.25 68.58) (xy 232.41 68.58))
-    (stroke (width 0) (type default) (color 0 0 0 0))
-  )
   (wire (pts (xy 222.25 38.1) (xy 232.41 38.1))
     (stroke (width 0) (type default) (color 0 0 0 0))
@@
     (stroke (width 0) (type default) (color 0 0 0 0))
   )
-  (bus (pts (xy 219.71 68.58) (xy 219.71 71.12))
-    (stroke (width 0) (type default) (color 0 0 0 0))
-  )
   (bus (pts (xy 57.15 105.41) (xy 57.15 113.03))
     (stroke (width 0) (type default) (color 0 0 0 0))
@@
     (stroke (width 0) (type default) (color 0 0 0 0))
   )
-  (bus (pts (xy 219.71 92.71) (xy 269.24 92.71))
+  (bus (pts (xy 219.71 92.71) (xy 242.57 92.71))
     (stroke (width 0) (type default) (color 0 0 0 0))
   )
@@
     (stroke (width 0) (type default) (color 0 0 0 0))
   )
+  (wire (pts (xy 73.66 121.92) (xy 85.09 121.92))
+    (stroke (width 0) (type default) (color 0 0 0 0))
+  )
   (wire (pts (xy 222.25 35.56) (xy 232.41 35.56))
     (stroke (width 0) (type default) (color 0 0 0 0))
@@
     (stroke (width 0) (type default) (color 0 0 0 0))
   )
+  (wire (pts (xy 245.11 86.36) (xy 245.11 90.17))
+    (stroke (width 0) (type default) (color 0 0 0 0))
+  )
   (wire (pts (xy 57.15 45.72) (xy 57.15 48.26))
     (stroke (width 0) (type default) (color 0 0 0 0))
@@
     (effects (font (size 1.27 1.27)) (justify left bottom))
   )
+  (label "+5V" (at 166.37 25.4 0)
+    (effects (font (size 1.27 1.27)) (justify left bottom))
+  )
+  (label "GND" (at 189.23 90.17 90)
+    (effects (font (size 1.27 1.27)) (justify left bottom))
+  )
   (label "d0" (at 222.25 30.48 0)
     (effects (font (size 1.27 1.27)) (justify left bottom))
   )
   (label "+5V" (at 27.94 64.77 0)
-    (effects (font (size 1.27 1.27)) (justify left bottom))
-  )
-  (label "a1" (at 118.11 40.64 90)
     (effects (font (size 1.27 1.27)) (justify left bottom))
   )
@@
     (effects (font (size 1.27 1.27)) (justify left bottom))
   )
+  (label "tapeout" (at 128.27 90.17 90)
+    (effects (font (size 1.27 1.27)) (justify left bottom))
+  )
   (label "+5V" (at 27.94 38.1 0)
     (effects (font (size 1.27 1.27)) (justify left bottom))
@@
   )
   (label "d5" (at 222.25 43.18 0)
+    (effects (font (size 1.27 1.27)) (justify left bottom))
+  )
+  (label "wr" (at 90.17 60.96 0)
     (effects (font (size 1.27 1.27)) (justify left bottom))
   )
@@
     (effects (font (size 1.27 1.27)) (justify left bottom))
   )
+  (label "+5V" (at 222.25 25.4 0)
+    (effects (font (size 1.27 1.27)) (justify left bottom))
+  )
+  (label "GND" (at 222.25 55.88 0)
+    (effects (font (size 1.27 1.27)) (justify left bottom))
+  )
   (label "d0" (at 166.37 30.48 0)
     (effects (font (size 1.27 1.27)) (justify left bottom))
@@
     (effects (font (size 1.27 1.27)) (justify left bottom))
   )
+  (label "GND" (at 166.37 55.88 0)
+    (effects (font (size 1.27 1.27)) (justify left bottom))
+  )
+  (label "d1" (at 138.43 90.17 90)
+    (effects (font (size 1.27 1.27)) (justify left bottom))
+  )
   (label "d3" (at 135.89 40.64 90)
     (effects (font (size 1.27 1.27)) (justify left bottom))
@@
     (effects (font (size 1.27 1.27)) (justify left bottom))
   )
+  (label "a0" (at 82.55 121.92 180)
+    (effects (font (size 1.27 1.27)) (justify right bottom))
+  )
   (label "bdir" (at 90.17 66.04 0)
     (effects (font (size 1.27 1.27)) (justify left bottom))
@@
     (effects (font (size 1.27 1.27)) (justify left bottom))
   )
+  (label "beeper" (at 120.65 90.17 90)
+    (effects (font (size 1.27 1.27)) (justify left bottom))
+  )
   (label "GND" (at 27.94 72.39 0)
     (effects (font (size 1.27 1.27)) (justify left bottom))
@@
     (effects (font (size 1.27 1.27)) (justify left bottom))
   )
-  (label "wr" (at 92.71 48.26 180)
-    (effects (font (size 1.27 1.27)) (justify right bottom))
+  (label "a0" (at 90.17 58.42 0)
+    (effects (font (size 1.27 1.27)) (justify left bottom))
   )
   (label "wr" (at 44.45 146.05 0)
@@
     (effects (font (size 1.27 1.27)) (justify right bottom))
   )
+  (label "+5V" (at 222.25 63.5 0)
+    (effects (font (size 1.27 1.27)) (justify left bottom))
+  )
+  (label "GND" (at 245.11 90.17 90)
+    (effects (font (size 1.27 1.27)) (justify left bottom))
+  )
   (label "d4" (at 115.57 40.64 90)
     (effects (font (size 1.27 1.27)) (justify left bottom))
@@
     (effects (font (size 1.27 1.27)) (justify left bottom))
   )
+  (label "+5V" (at 166.37 63.5 0)
+    (effects (font (size 1.27 1.27)) (justify left bottom))
+  )
   (label "reset" (at 222.25 71.12 0)
     (effects (font (size 1.27 1.27)) (justify left bottom))
@@
     (effects (font (size 1.27 1.27)) (justify left bottom))
   )
-  (label "d1" (at 157.48 55.88 180)
-    (effects (font (size 1.27 1.27)) (justify right bottom))
-  )
   (label "d2" (at 45.72 120.65 0)

Commit message: >> прототип на макетке поет
Parts:
- added C10, C9: 0.47uF wima, Capacitor_THT:C_Rect_L7.0mm_W2.5mm_P5.00mm, symbol Device:C
- added C11: 0.47uF50VX7R0805, Capacitor_SMD:C_0805_2012Metric_Pad1.18x1.45mm_HandSolder, symbol Device:C
- added Q1: BC847, Package_TO_SOT_SMD:SOT-23, symbol Transistor_BJT:BC847
- added R10, R9: 1K, Resistor_SMD:R_0805_2012Metric_Pad1.20x1.40mm_HandSolder, symbol Device:R
- added R11, R12, R13, R14, R15, R16, R2, R3, R6, R7: 10K, Resistor_SMD:R_0805_2012Metric_Pad1.20x1.40mm_HandSolder, symbol Device:R
- added R4, R5, R8: 4.7K, Resistor_SMD:R_0805_2012Metric_Pad1.20x1.40mm_HandSolder, symbol Device:R
- R1: value 1K -> 4.7K
- U2: renamed from U4; footprint (none) -> Package_DIP:DIP-8_W7.62mm_Socket
- renumbered C9 to C12, C10 to C13, C3 to C2, C4 to C3, C5 to C4, C6 to C5, C2 to C6, U3 to U1, U1 to U3, U2 to U4
Connections:
- net +5V: now also U2.8 (V+), Q1.3 (C), R16.1
- net GND: now also U2.4 (V-), C11.2, R10.1, R14.1, R9.1
- net reset: now also D1.4 (io)
- net YM_0_A: now reaches R1.1
- net YM_0_A: now also U3.3 (A)
- net at R1.2: now also C9.1, R2.2, R5.2, R6.2, R9.2
- net YM_0_C: now reaches U3.38 (C)
- net YM_0_C: now also R4.1
- net YM_0_B: now reaches U3.4 (B)
- net YM_0_B: now also R2.1, R3.1
- net at C13.2: now also U2.7, R15.2
- net at C12.1: now also U2.1, R13.2
- net YM_1_A: now reaches U4.3 (A)
- net YM_1_A: now also R5.1
- net YM_1_C: now reaches U4.38 (C)
- net YM_1_C: now also R8.1
- net YM_1_B: now reaches U4.4 (B)
- net YM_1_B: now also R6.1, R7.1
- net ioge_c: now reaches D1.27 (io)
- net ioge_c: now also Q1.1 (B)
- net IOGE: now reaches X1.44 (IOGE)
- net IOGE: now also Q1.2 (E)
- net at U2.2 (-): now also R11.2, R13.1
- net at U2.3 (+): now also U2.5 (+), C11.1, R14.2, R16.2
- net at U2.6 (-): now also R12.2, R15.1
- new net: C10.1, R12.1
- new net: C10.2, R10.2, R3.2, R4.2, R7.2, R8.2
- new net: C9.2, R11.1
Other:
- moved on the sheet: C12, C13, U2A, U2B
