File: sch_and_pcb/epm3032_ym2149x2.kicad_pcb (KiCad board)
At the start: 2 copper layers, 101.6 x 98.4 mm, 17 parts, among them U1 YM2149, U2 YM2149, U3 AMS1117-3.3, U4 NE5532, X1 zx-bus

Commit message: >> продолжаем продолжать. Макетка рулез.
Connections:
- D1 pad 11: unconnected-(D1-Pad11) -> /a0
- D1 pad 12: unconnected-(D1-Pad12) -> /wr
- D1 pad 21: unconnected-(D1-Pad21) -> /beeper
- D1 pad 28: unconnected-(D1-Pad28) -> /d1
- D1 pad 36: /d1 -> unconnected-(D1-Pad36)
- D1 pad 4: /a1 -> unconnected-(D1-Pad4)
- D1 pad 7: /wr -> unconnected-(D1-Pad7)
- U1 pad 1: unconnected-(U1-Pad1) -> /GND
- U1 pad 24: unconnected-(U1-Pad24) -> /GND
- U1 pad 28: unconnected-(U1-Pad28) -> /+5V
- U1 pad 40: unconnected-(U1-Pad40) -> /+5V
- U2 pad 1: unconnected-(U2-Pad1) -> /GND
- U2 pad 24: unconnected-(U2-Pad24) -> /GND
- U2 pad 28: unconnected-(U2-Pad28) -> /+5V
- U2 pad 40: unconnected-(U2-Pad40) -> /+5V
- X1 pad 40: unconnected-(X1-Pad40) -> /a0

Commit message: >> прототип на макетке поет
Parts:
- added C11: 0.47uF50VX7R0805, Capacitor_SMD:C_0805_2012Metric_Pad1.18x1.45mm_HandSolder, F.Cu at (71.4, 43.9)
- added C12: 0.47uF wima, Capacitor_THT:C_Rect_L7.0mm_W2.5mm_P5.00mm, F.Cu at (108.0, 51.1)
- added C13: 0.47uF wima, Capacitor_THT:C_Rect_L7.0mm_W2.5mm_P5.00mm, F.Cu at (108.0, 47.0)
- added Q1: BC847, Package_TO_SOT_SMD:SOT-23, F.Cu at (69.3, 114.6)
- added R10: 1K, Resistor_SMD:R_0805_2012Metric_Pad1.20x1.40mm_HandSolder, F.Cu at (97.0, 62.0)
- added R11: 10K, Resistor_SMD:R_0805_2012Metric_Pad1.20x1.40mm_HandSolder, F.Cu at (105.9, 59.4)
- added R12: 10K, Resistor_SMD:R_0805_2012Metric_Pad1.20x1.40mm_HandSolder, F.Cu at (106.0, 35.3)
- added R13: 10K, Resistor_SMD:R_0805_2012Metric_Pad1.20x1.40mm_HandSolder, F.Cu at (106.7, 65.5)
- added R14: 10K, Resistor_SMD:R_0805_2012Metric_Pad1.20x1.40mm_HandSolder, F.Cu at (71.4, 48.5)
- added R15: 10K, Resistor_SMD:R_0805_2012Metric_Pad1.20x1.40mm_HandSolder, F.Cu at (110.7, 81.3)
- added R16: 10K, Resistor_SMD:R_0805_2012Metric_Pad1.20x1.40mm_HandSolder, F.Cu at (71.4, 38.9)
- added R2: 10K, Resistor_SMD:R_0805_2012Metric_Pad1.20x1.40mm_HandSolder, F.Cu at (115.3, 80.5)
- added R3: 10K, Resistor_SMD:R_0805_2012Metric_Pad1.20x1.40mm_HandSolder, F.Cu at (110.7, 86.9)
- added R4: 4.7K, Resistor_SMD:R_0805_2012Metric_Pad1.20x1.40mm_HandSolder, F.Cu at (120.4, 85.3)
- added R5: 4.7K, Resistor_SMD:R_0805_2012Metric_Pad1.20x1.40mm_HandSolder, F.Cu at (116.3, 101.1)
- added R6: 10K, Resistor_SMD:R_0805_2012Metric_Pad1.20x1.40mm_HandSolder, F.Cu at (110.7, 100.1)
- added R7: 10K, Resistor_SMD:R_0805_2012Metric_Pad1.20x1.40mm_HandSolder, F.Cu at (111.0, 104.9)
- added R8: 4.7K, Resistor_SMD:R_0805_2012Metric_Pad1.20x1.40mm_HandSolder, F.Cu at (118.4, 107.7)
- added R9: 1K, Resistor_SMD:R_0805_2012Metric_Pad1.20x1.40mm_HandSolder, F.Cu at (90.9, 66.8)
- R1: value 1K -> 4.7K
- U1: value YM2149 -> AMS1117-3.3; footprint Package_DIP:DIP-40_W15.24mm -> Package_TO_SOT_SMD:SOT-223-3_TabPin2
- U2: value YM2149 -> NE5532; footprint Package_DIP:DIP-40_W15.24mm -> Package_DIP:DIP-8_W7.62mm_Socket
- U3: value AMS1117-3.3 -> YM2149; footprint Package_TO_SOT_SMD:SOT-223-3_TabPin2 -> Package_DIP:DIP-40_W15.24mm
- U4: value NE5532 -> YM2149; footprint Package_SO:SOIC-8_3.9x4.9mm_P1.27mm -> Package_DIP:DIP-40_W15.24mm
- moved U3 91.2 mm to (122.2, 75.7), turned to -90 degrees
- moved U4 78.8 mm to (122.2, 96.0), turned to -90 degrees
- moved R1 75.4 mm to (120.4, 69.1)
- moved U1 45.9 mm to (33.8, 94.7)
- moved C9 43.4 mm to (116.9, 59.4)
- moved U2 22.2 mm to (67.8, 57.9)
- moved D1 9.20 mm to (60.2, 103.6), turned to -90 degrees
Connections:
- C10 pad 1: unconnected-(C10-Pad1) -> Net-(C10-Pad1)
- C10 pad 2: unconnected-(C10-Pad2) -> Net-(C10-Pad2)
- C3 pad 1: /+3.3V -> /+5V
- C4 pad 1: /+5V -> /+3.3V
- C5 pad 1: /+3.3V -> /+5V
- C6 pad 1: /+5V -> /+3.3V
- C9 pad 1: unconnected-(C9-Pad1) -> Net-(C9-Pad1)
- C9 pad 2: unconnected-(C9-Pad2) -> Net-(C9-Pad2)
- D1 pad 24: unconnected-(D1-Pad24) -> /tapeout
- D1 pad 27: unconnected-(D1-Pad27) -> /ioge_c
- D1 pad 4: unconnected-(D1-Pad4) -> /reset
- R1 pad 1: unconnected-(R1-Pad1) -> /YM_0_A
- R1 pad 2: unconnected-(R1-Pad2) -> Net-(C9-Pad1)
- U1 pad 2: unconnected-(U1-Pad2) -> /+3.3V
- U1 pad 3: unconnected-(U1-Pad3) -> /+5V
- U2 pad 1: /GND -> Net-(C12-Pad1)
- U2 pad 2: unconnected-(U2-Pad2) -> Net-(R11-Pad2)
- U2 pad 3: unconnected-(U2-Pad3) -> Net-(C11-Pad1)
- U2 pad 4: unconnected-(U2-Pad4) -> /GND
- U2 pad 5: unconnected-(U2-Pad5) -> Net-(C11-Pad1)
- U2 pad 6: unconnected-(U2-Pad6) -> Net-(R12-Pad2)
- U2 pad 7: unconnected-(U2-Pad7) -> Net-(C13-Pad2)
- U2 pad 8: unconnected-(U2-Pad8) -> /+5V
- U3 pad 2: /+3.3V -> unconnected-(U3-Pad2)
- U3 pad 3: /+5V -> /YM_0_A
- U4 pad 1: unconnected-(U4-Pad1) -> /GND
- U4 pad 3: unconnected-(U4-Pad3) -> /YM_1_A
- U4 pad 4: unconnected-(U4-Pad4) -> /YM_1_B
- X1 pad 44: unconnected-(X1-Pad44) -> /IOGE

Commit message: >> добавил сигнал dos, нужно тестировать.
Parts:
- added U5: 74HC374, Package_DIP:DIP-20_W7.62mm, F.Cu at (57.7, 64.3)
- added U7: AD7533JN, Package_DIP:DIP-16_W7.62mm, F.Cu at (34.1, 64.3)
- U2: value NE5532 -> LM324; footprint Package_DIP:DIP-8_W7.62mm_Socket -> Package_DIP:DIP-14_W7.62mm
- moved U2 29.4 mm to (53.1, 32.5)
- moved C7 15.0 mm to (50.5, 80.8)
- moved C3 15.0 mm to (50.5, 75.7)
- moved C1 10.5 mm to (62.8, 82.5)
- moved C4 10.5 mm to (62.8, 77.5)
- moved C8 10.5 mm to (62.8, 87.6)
- renumbered U3 to U4, U4 to U6
Connections:
- D1 pad 37: /d2 -> /int
- U2 pad 1: Net-(C12-Pad1) -> unconnected-(U2-Pad1)
- U2 pad 2: Net-(R11-Pad2) -> unconnected-(U2-Pad2)
- U2 pad 3: Net-(C11-Pad1) -> unconnected-(U2-Pad3)
- U2 pad 4: /GND -> /+5V
- U2 pad 5: Net-(C11-Pad1) -> unconnected-(U2-Pad5)
- U2 pad 6: Net-(R12-Pad2) -> unconnected-(U2-Pad6)
- U2 pad 7: Net-(C13-Pad2) -> unconnected-(U2-Pad7)
- U2 pad 8: /+5V -> Net-(C12-Pad1)
